File: Microwave_LO_Generator/frequencySynthesizer.sch (KiCad schematic (older format))
At the start: 28 parts, among them J4 Conn_01x05_Male, U1 ADF4150HV, X1 IQXT-220-1

Commit message: backup
Parts:
- C1, C11, C12, C8: Manufacturer/Part Number GRM1555C2A100GA01D -> 04025A100JAT2A; Supplier Stock Code Mouser 81-GRM1555C2A100GA1D -> 581-04025A100J
- C10: Manufacturer/Part Number C0402C104J8RACAUTO -> 963-GMK105CC6105MV-F; Supplier Stock Code Mouser 80-C0402C104J8RAUTO -> GMK105CC6105MV-F
- C13: Manufacturer/Part Number GCM155R71H331KA37J -> GRM022R71C331KE14L; Supplier Stock Code Mouser 881-GCM155R71H331KA7J -> 81-GRM022R71C331KE4L
- C14: Supplier Stock Code Mouser 81-GCM155R71H562JA5D -> 81-GCM155R71H562JA5D
- C15: Manufacturer/Part Number GCM1555C1H121JA16D -> 04023A121JAT2A; Supplier Stock Code Mouser 81-GCM1555C1H121JA6D -> 581-04023A121JAT2A
- C2, C7, C9: Manufacturer/Part Number C0402C104J8RACAUTO -> 581-0402YD104MAT2A; Supplier Stock Code Mouser 80-C0402C104J8RAUTO -> 0402YD104MAT2A
- C4: Manufacturer/Part Number GRM1555C1H102FA01D -> 04025C102JAT2A; Supplier Stock Code Mouser 81-GRM1555C1H102FA1D -> 581-04025C102J
- C6: Supplier Stock Code Mouser 81-GCM1555C1H101JA6D -> 81-GCM1555C1H101JA6D
- D1: Supplier Stock Code Mouser 630-HSMG-C170 -> 630-HSMG-C170
Changed lines of the file:
@@
 F 2 "Capacitor_SMD:C_0402_1005Metric_Pad0.74x0.62mm_HandSolder" H 4988 2700 50  0001 C CNN
 F 3 "~" H 4950 2850 50  0001 C CNN
-F 4 "GRM1555C2A100GA01D" H 4950 2850 50  0001 C CNN "Manufacturer/Part Number"
-F 5 "Mouser 81-GRM1555C2A100GA1D" H 4950 2850 50  0001 C CNN "Supplier Stock Code"
+F 4 "04025A100JAT2A" H 4950 2850 50  0001 C CNN "Manufacturer/Part Number"
+F 5 "581-04025A100J" H 4950 2850 50  0001 C CNN "Supplier Stock Code"
 	1    4950 2850
 	-1   0    0    1
@@
 F 2 "Capacitor_SMD:C_0402_1005Metric_Pad0.74x0.62mm_HandSolder" H 4588 2700 50  0001 C CNN
 F 3 "~" H 4550 2850 50  0001 C CNN
-F 4 "Mouser 80-C0402C104J8RAUTO" H 4550 2850 50  0001 C CNN "Supplier Stock Code"
-F 5 "C0402C104J8RACAUTO" H 4550 2850 50  0001 C CNN "Manufacturer/Part Number"
+F 4 "0402YD104MAT2A" H 4550 2850 50  0001 C CNN "Supplier Stock Code"
+F 5 "581-0402YD104MAT2A" H 4550 2850 50  0001 C CNN "Manufacturer/Part Number"
 	1    4550 2850
 	-1   0    0    1
@@
 F 2 "Capacitor_SMD:C_0402_1005Metric_Pad0.74x0.62mm_HandSolder" H 5788 2700 50  0001 C CNN
 F 3 "~" H 5750 2850 50  0001 C CNN
-F 4 "Mouser 80-C0402C104J8RAUTO" H 5750 2850 50  0001 C CNN "Supplier Stock Code"
-F 5 "C0402C104J8RACAUTO" H 5750 2850 50  0001 C CNN "Manufacturer/Part Number"
+F 4 "0402YD104MAT2A" H 5750 2850 50  0001 C CNN "Supplier Stock Code"
+F 5 "581-0402YD104MAT2A" H 5750 2850 50  0001 C CNN "Manufacturer/Part Number"
 	1    5750 2850
 	-1   0    0    1
@@
 F 2 "Capacitor_SMD:C_0402_1005Metric_Pad0.74x0.62mm_HandSolder" H 6188 2700 50  0001 C CNN
 F 3 "~" H 6150 2850 50  0001 C CNN
-F 4 "GRM1555C2A100GA01D" H 6150 2850 50  0001 C CNN "Manufacturer/Part Number"
-F 5 "Mouser 81-GRM1555C2A100GA1D" H 6150 2850 50  0001 C CNN "Supplier Stock Code"
+F 4 "04025A100JAT2A" H 6150 2850 50  0001 C CNN "Manufacturer/Part Number"
+F 5 "581-04025A100J" H 6150 2850 50  0001 C CNN "Supplier Stock Code"
 	1    6150 2850
 	-1   0    0    1
@@
 F 2 "Capacitor_SMD:C_0402_1005Metric_Pad0.74x0.62mm_HandSolder" H 1738 3000 50  0001 C CNN
 F 3 "~" H 1700 3150 50  0001 C CNN
-F 4 "Mouser 80-C0402C104J8RAUTO" H 1700 3150 50  0001 C CNN "Supplier Stock Code"
-F 5 "C0402C104J8RACAUTO" H 1700 3150 50  0001 C CNN "Manufacturer/Part Number"
+F 4 "0402YD104MAT2A" H 1700 3150 50  0001 C CNN "Supplier Stock Code"
+F 5 "581-0402YD104MAT2A" H 1700 3150 50  0001 C CNN "Manufacturer/Part Number"
 	1    1700 3150
 	-1   0    0    1
@@
 F 2 "Capacitor_SMD:C_0402_1005Metric_Pad0.74x0.62mm_HandSolder" H 1338 3000 50  0001 C CNN
 F 3 "~" H 1300 3150 50  0001 C CNN
-F 4 "GRM1555C2A100GA01D" H 1300 3150 50  0001 C CNN "Manufacturer/Part Number"
-F 5 "Mouser 81-GRM1555C2A100GA1D" H 1300 3150 50  0001 C CNN "Supplier Stock Code"
+F 4 "04025A100JAT2A" H 1300 3150 50  0001 C CNN "Manufacturer/Part Number"
+F 5 "581-04025A100J" H 1300 3150 50  0001 C CNN "Supplier Stock Code"
 	1    1300 3150
 	-1   0    0    1
@@
 F 2 "Capacitor_SMD:C_0402_1005Metric_Pad0.74x0.62mm_HandSolder" H 3538 3950 50  0001 C CNN
 F 3 "~" H 3500 4100 50  0001 C CNN
-F 4 "GRM1555C1H102FA01D" H 3500 4100 50  0001 C CNN "Manufacturer/Part Number"
-F 5 "Mouser 81-GRM1555C1H102FA1D" H 3500 4100 50  0001 C CNN "Supplier Stock Code"
+F 4 "04025C102JAT2A" H 3500 4100 50  0001 C CNN "Manufacturer/Part Number"
+F 5 "581-04025C102J" H 3500 4100 50  0001 C CNN "Supplier Stock Code"
 	1    3500 4100
 	0    1    1    0
@@
 F 2 "Capacitor_SMD:C_0402_1005Metric_Pad0.74x0.62mm_HandSolder" H 6638 3700 50  0001 C CNN
 F 3 "~" H 6600 3850 50  0001 C CNN
-F 4 "GCM155R71H331KA37J" H 6600 3850 50  0001 C CNN "Manufacturer/Part Number"
-F 5 "Mouser 881-GCM155R71H331KA7J" H 6600 3850 50  0001 C CNN "Supplier Stock Code"
+F 4 "GRM022R71C331KE14L" H 6600 3850 50  0001 C CNN "Manufacturer/Part Number"
+F 5 "81-GRM022R71C331KE4L" H 6600 3850 50  0001 C CNN "Supplier Stock Code"
 	1    6600 3850
 	-1   0    0    1
@@
 F 3 "~" H 7050 4050 50  0001 C CNN
 F 4 "GCM155R71H562JA55D" H 7050 4050 50  0001 C CNN "Manufacturer/Part Number"
-F 5 "Mouser 81-GCM155R71H562JA5D" H 7050 4050 50  0001 C CNN "Supplier Stock Code"
+F 5 "81-GCM155R71H562JA5D" H 7050 4050 50  0001 C CNN "Supplier Stock Code"
 	1    7050 4050
 	-1   0    0    1
@@
 F 2 "Capacitor_SMD:C_0402_1005Metric_Pad0.74x0.62mm_HandSolder" H 7788 3600 50  0001 C CNN
 F 3 "~" H 7750 3750 50  0001 C CNN
-F 4 "GCM1555C1H121JA16D" H 7750 3750 50  0001 C CNN "Manufacturer/Part Number"
-F 5 "Mouser 81-GCM1555C1H121JA6D" H 7750 3750 50  0001 C CNN "Supplier Stock Code"
+F 4 "04023A121JAT2A" H 7750 3750 50  0001 C CNN "Manufacturer/Part Number"
+F 5 "581-04023A121JAT2A" H 7750 3750 50  0001 C CNN "Supplier Stock Code"
 	1    7750 3750
 	-1   0    0    1
@@
 F 3 "https://www.mouser.it/datasheet/2/678/av02-0551en-ds-hsmx-cxxx-05mar2012-1827675.pdf" H 6900 5000 50  0001 C CNN
 F 4 "HSMG-C170" H 6900 5000 50  0001 C CNN "Manufacturer/Part Number"
-F 5 "Mouser 630-HSMG-C170" H 6900 5000 50  0001 C CNN "Supplier Stock Code"
+F 5 "630-HSMG-C170" H 6900 5000 50  0001 C CNN "Supplier Stock Code"
 	1    6900 5000
 	0    -1   -1   0
@@
 F 3 "~" H 4300 5300 50  0001 C CNN
 F 4 "GCM1555C1H101JA16D" H 4300 5300 50  0001 C CNN "Manufacturer/Part Number"
-F 5 "Mouser 81-GCM1555C1H101JA6D" H 4300 5300 50  0001 C CNN "Supplier Stock Code"
+F 5 "81-GCM1555C1H101JA6D" H 4300 5300 50  0001 C CNN "Supplier Stock Code"
 	1    4300 5300
 	-1   0    0    1
@@
 F 2 "Capacitor_SMD:C_0402_1005Metric_Pad0.74x0.62mm_HandSolder" H 5888 2050 50  0001 C CNN
 F 3 "~" H 5850 2200 50  0001 C CNN
-F 4 "Mouser 80-C0402C104J8RAUTO" H 5850 2200 50  0001 C CNN "Supplier Stock Code"
-F 5 "C0402C104J8RACAUTO" H 5850 2200 50  0001 C CNN "Manufacturer/Part Number"
+F 4 "GMK105CC6105MV-F" H 5850 2200 50  0001 C CNN "Supplier Stock Code"
+F 5 "963-GMK105CC6105MV-F" H 5850 2200 50  0001 C CNN "Manufacturer/Part Number"
 	1    5850 2200
 	-1   0    0    1
@@
 F 2 "Capacitor_SMD:C_0402_1005Metric_Pad0.74x0.62mm_HandSolder" H 6288 2050 50  0001 C CNN
 F 3 "~" H 6250 2200 50  0001 C CNN
-F 4 "GRM1555C2A100GA01D" H 6250 2200 50  0001 C CNN "Manufacturer/Part Number"
-F 5 "Mouser 81-GRM1555C2A100GA1D" H 6250 2200 50  0001 C CNN "Supplier Stock Code"
+F 4 "04025A100JAT2A" H 6250 2200 50  0001 C CNN "Manufacturer/Part Number"
+F 5 "581-04025A100J" H 6250 2200 50  0001 C CNN "Supplier Stock Code"
 	1    6250 2200
 	-1   0    0    1

Commit message: update bom
Parts:
- U1: Supplier Stock Code Mouser 584-ADF4150HVBCPZ -> 584-ADF4150HVBCPZ
- X1: Manufacturer/Part Number (none) -> IQXT-220-1; Supplier Stock Code (none) -> LFTCXO075792Cutt
- renumbered C12 to C10, C13 to C11, C14 to C12, C15 to C13, C4 to C3, C6 to C4, C7 to C5, C8 to C6, C9 to C7, C10 to C8, C11 to C9, J4 to J1, R10 to R1, R6 to R10, R1 to R2, R18 to R3, R19 to R4, R20 to R5, R2 to R6, R3 to R7, R4 to R8, R5 to R9

Commit message: Update for DRC
Parts:
- J1: footprint Connector_PinHeader_2.54mm:PinHeader_1x05_P2.54mm_Vertical -> Microwave_LO_Generator:PinHeader_1x05_P2.54mm_Vertical
- TP1: footprint TestPoint:TestPoint_Loop_D2.60mm_Drill1.6mm_Beaded -> Microwave_LO_Generator:TestPoint_Loop_D2.60mm_Drill1.6mm_Beaded
- X1: footprint Oscillator:Oscillator_SMD_Abracon_ASE-4Pin_3.2x2.5mm_HandSoldering -> Microwave_LO_Generator:Oscillator_SMD_Abracon_ASE-4Pin_3.2x2.5mm_HandSoldering
Changed lines of the file:
@@
 F 0 "X1" H 2544 3596 50  0000 L CNN
 F 1 "IQXT-220-1" H 2544 3505 50  0000 L CNN
-F 2 "Oscillator:Oscillator_SMD_Abracon_ASE-4Pin_3.2x2.5mm_HandSoldering" H 2200 3550 50  0001 C CNN
+F 2 "Microwave_LO_Generator:Oscillator_SMD_Abracon_ASE-4Pin_3.2x2.5mm_HandSoldering" H 2200 3550 50  0001 C CNN
 F 3 "https://www.mouser.it/datasheet/2/741/LFTCXO075792Cutt-1115708.pdf" H 2200 3550 50  0001 C CNN
 F 4 "IQXT-220-1" H 2200 3550 50  0001 C CNN "Manufacturer/Part Number"
@@
 F 0 "TP1" H 3092 3476 50  0000 R CNN
 F 1 "TestPoint" H 3092 3567 50  0000 R CNN
-F 2 "TestPoint:TestPoint_Loop_D2.60mm_Drill1.6mm_Beaded" H 3350 3450 50  0001 C CNN
+F 2 "Microwave_LO_Generator:TestPoint_Loop_D2.60mm_Drill1.6mm_Beaded" H 3350 3450 50  0001 C CNN
 F 3 "https://www.mouser.it/datasheet/2/215/005-5009-741293.pdf" H 3350 3450 50  0001 C CNN
 F 4 "5007" H 3150 3450 50  0001 C CNN "Manufacturer/Part Number"
@@
 F 0 "J1" H 2858 2181 50  0000 C CNN
 F 1 "Conn_01x05_Male" H 2858 2090 50  0000 C CNN
-F 2 "Connector_PinHeader_2.54mm:PinHeader_1x05_P2.54mm_Vertical" H 2750 1800 50  0001 C CNN
+F 2 "Microwave_LO_Generator:PinHeader_1x05_P2.54mm_Vertical" H 2750 1800 50  0001 C CNN
 F 3 "~" H 2750 1800 50  0001 C CNN
 	1    2750 1800
